File: Projekt/Projekt.kicad_pcb (KiCad board)
At the start: 2 copper layers, 7 parts, among them U1 SHT4x, U2 STM32F446RETx, U3 AMS1117-3.3, U4 PCF8574AP

Commit message: Update
Parts:
- removed RV1: R_Potentiometer_Small, Potentiometer_THT:Potentiometer_Bourns_3299Y_Vertical
- added C1: 100n, Capacitor_SMD:C_0402_1005Metric, F.Cu at (142.2, 93.1)
- added C10: 22u, Capacitor_SMD:C_0805_2012Metric, F.Cu at (154.5, 111.0)
- added C11: 22u, Capacitor_SMD:C_0805_2012Metric, F.Cu at (126.8, 103.0)
- added C2: 100n, Capacitor_SMD:C_0402_1005Metric, F.Cu at (126.2, 97.9)
- added C3: 100n, Capacitor_SMD:C_0402_1005Metric, F.Cu at (143.0, 107.8)
- added C4: 100n, Capacitor_SMD:C_0402_1005Metric, F.Cu at (147.0, 95.2)
- added C5: 10u, Capacitor_SMD:C_0402_1005Metric, F.Cu at (147.2, 108.6)
- added C6: 10n, Capacitor_SMD:C_0402_1005Metric, F.Cu at (144.8, 110.8)
- added C7: 1u, Capacitor_SMD:C_0402_1005Metric, F.Cu at (144.8, 96.8)
- added C8: 1u, Capacitor_SMD:C_0402_1005Metric, F.Cu at (152.0, 94.4)
- added C9: 100n, Capacitor_SMD:C_0402_1005Metric, F.Cu at (128.5, 99.5)
- added D1: LED, LED_SMD:LED_0603_1608Metric, F.Cu at (121.8, 104.2)
- added FB1: 120 R, Inductor_SMD:L_0603_1608Metric, F.Cu at (146.5, 93.5)
- added H1: MountingHole, MountingHole:MountingHole_3mm, F.Cu at (69.8, 82.5)
- added H2: MountingHole, MountingHole:MountingHole_3mm, F.Cu at (163.0, 91.0)
- added H3: MountingHole, MountingHole:MountingHole_3mm, F.Cu at (163.0, 114.5)
- added H4: MountingHole, MountingHole:MountingHole_3mm, F.Cu at (88.2, 112.8)
- added J1: USB_B_Micro, Connector_USB:USB_Micro-B_Wuerth_629105150521, F.Cu at (161.2, 103.3)
- added J2: Conn_01x04_Pin, Connector_PinHeader_2.54mm:PinHeader_1x04_P2.54mm_Vertical, F.Cu at (133.8, 89.9)
- added R1: 10k, Resistor_SMD:R_0402_1005Metric, F.Cu at (121.2, 98.0)
- added R2: 1k5, Resistor_SMD:R_0402_1005Metric, F.Cu at (124.0, 100.0)
- added SW1: SW_SPDT, Button_Switch_THT:SW_E-Switch_EG1224_SPDT_Angled, F.Cu at (116.1, 103.8)
- R3: footprint Resistor_SMD:R_1206_3216Metric_Pad1.30x1.75mm_HandSolder -> Resistor_SMD:R_0402_1005Metric
- moved U4 107.8 mm to (140.0, 108.9), turned to -90 degrees
- moved R3 99.4 mm to (147.8, 116.0), turned to -90 degrees
- moved U3 97.0 mm to (151.0, 103.2), turned to -90 degrees
- moved DS1 72.8 mm to (93.5, 120.9)
- moved U1 52.4 mm to (148.6, 111.7), turned to 90 degrees
- moved U2 17.0 mm to (136.2, 99.8)
Connections:
- DS1 pad 3: Net-(DS1-VO) -> unconnected-(DS1-VO-Pad3)
Routing:
- added copper zone on B.Cu, net GND
Other:
- board outline added: 83.1 x 68.6 mm

Commit message: Final
Parts:
- H1, H2, H3, H4: footprint MountingHole:MountingHole_3mm -> MountingHole:MountingHole_2mm
- moved H4 88.2 mm to (164.2, 157.7)
- moved H3 87.5 mm to (86.9, 157.8)
- moved H1 71.6 mm to (140.1, 96.0)
- moved H2 68.7 mm to (94.5, 96.0)
- moved U4 46.4 mm to (94.3, 116.8), turned to 90 degrees
- moved C8 34.9 mm to (118.5, 104.1), turned to -90 degrees
- moved C4 34.8 mm to (119.1, 116.0), turned to -90 degrees
- moved C7 33.0 mm to (116.9, 114.5), turned to -90 degrees
- moved C10 31.0 mm to (125.3, 100.7), turned to 0 degrees
- moved FB1 29.1 mm to (118.5, 101.5), turned to -90 degrees
- moved J2 26.6 mm to (115.6, 109.2), turned to 180 degrees
- moved C6 24.6 mm to (122.1, 101.2), turned to 0 degrees
- moved J1 24.2 mm to (137.0, 103.6), turned to -90 degrees
- moved C1 24.2 mm to (134.2, 116.0)
- moved C5 22.7 mm to (126.2, 117.3), turned to 180 degrees
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Connections:
- U2 pad 23: unconnected-(U2-PA7-Pad23) -> Net-(U1-SCL)
- U2 pad 41: Net-(U1-SCL) -> unconnected-(U2-PA8-Pad41)
Routing:
- net 5V USB: track 0.00 -> 90.0 mm
- net GND: track 0.00 -> 83.8 mm, vias 0 -> 7
- net 3V3: track 0.00 -> 79.7 mm
- net Net-(DS1-D7): track 0.00 -> 33.2 mm
- net Net-(U2-PB7): track 0.00 -> 31.0 mm
- net Net-(DS1-D6): track 0.00 -> 27.7 mm
- net Net-(U2-PB6): track 0.00 -> 22.3 mm
- net Net-(DS1-D5): track 0.00 -> 22.2 mm
- net Net-(J1-D+): track 0.00 -> 18.8 mm
- net Net-(J1-D-): track 0.00 -> 17.2 mm
- net Net-(SW1-B): track 0.00 -> 16.0 mm, vias 0 -> 2
- net Net-(DS1-D4): track 0.00 -> 15.6 mm
- net Net-(J2-Pin_3): track 0.00 -> 11.9 mm, vias 0 -> 2
- net Net-(DS1-LED(+)): track 0.00 -> 5.13 mm
- net Net-(U1-SDA): track 0.00 -> 5.05 mm
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Other:
- board size 83.1 x 68.6 mm -> 82.1 x 66.8 mm

Commit message: Final
Parts:
- moved J1 0.10 mm to (136.9, 103.6), turned to 90 degrees
Routing:
- net Net-(J1-D+): track 18.8 -> 14.1 mm
- net Net-(J1-D-): track 17.2 -> 14.8 mm
- net 5V USB: track 90.0 -> 91.0 mm
