File: Projekt/Projekt.kicad_sch (KiCad schematic)
At the start: 25 parts, among them J1 USB_B_Micro, J2 Conn_01x04_Pin, SW1 SW_SPDT, U1 SHT4x, U2 STM32F446RETx, U3 AMS1117-3.3, U4 PCF8574AP

Commit message: Update
Parts:
- removed RV1: R_Potentiometer_Small, Potentiometer_THT:Potentiometer_Bourns_3299Y_Vertical, symbol Device:R_Potentiometer_Small
- added H1, H2, H3, H4: MountingHole, MountingHole:MountingHole_3mm, symbol Mechanical:MountingHole
- C1, C2, C3, C4, C5, C6, C7, C8, C9: footprint (none) -> Capacitor_SMD:C_0402_1005Metric
- C10, C11: footprint (none) -> Capacitor_SMD:C_0805_2012Metric
- D1: footprint (none) -> LED_SMD:LED_0603_1608Metric
- FB1: footprint (none) -> Inductor_SMD:L_0603_1608Metric
- J1: footprint (none) -> Connector_USB:USB_Micro-B_Wuerth_629105150521
- J2: footprint (none) -> Connector_PinHeader_2.54mm:PinHeader_1x04_P2.54mm_Vertical
- R1, R2: footprint (none) -> Resistor_SMD:R_0402_1005Metric
- R3: footprint Resistor_SMD:R_1206_3216Metric_Pad1.30x1.75mm_HandSolder -> Resistor_SMD:R_0402_1005Metric
- SW1: footprint (none) -> Button_Switch_THT:SW_E-Switch_EG1224_SPDT_Angled
Connections:
- no-connect marks 51 -> 52
Other:
- moved on the sheet: R3

Commit message: Final
Parts:
- H1, H2, H3, H4: footprint MountingHole:MountingHole_3mm -> MountingHole:MountingHole_2mm
Connections:
- net at U1.2 (SCL): now also U2.23 (PA7); no longer U2.41 (PA8)
Other:
- note added: "AMS1117 REGULATOR"
- note added: "STM32F446RE, LCD i SHT4X"
- moved on the sheet: C1, C10, C11, C2, C3, C4, C5, C6, C7, C8, C9, D1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
